Commit message: implementation de moveit avec simulateur Sycobot

File: dsr_description/urdf/m1013.urdf (robot description, URDF)
Before this commit: robot m1013, 8 links, 7 joints
Links:
- removed link base
Joints:
- removed joint fixed

File: dsr_description/xacro/macro.m1013.blue.xacro (robot description, xacro)
@@ -1,9 +1,9 @@
 <?xml version="1.0"?>
 <robot name="m1013" xmlns:xacro="http://www.ros.org/wiki/xacro">
-	<xacro:include filename="$(find dsr_description)/config/macro.gazebo.xacro" />
-	<xacro:include filename="$(find dsr_description)/config/macro.transmission.xacro" />
-	<xacro:include filename="$(find dsr_description)/config/macro.materials.xacro" />
+<!--	<xacro:include filename="$(find dsr_description)/config/macro.gazebo.xacro" />-->
+<!--	<xacro:include filename="$(find dsr_description)/config/macro.transmission.xacro" />-->
+<!--	<xacro:include filename="$(find dsr_description)/config/macro.materials.xacro" />-->
 	<xacro:macro name="m1013" params="namespace">
-		<xacro:dsr_materials />
+<!--		<xacro:dsr_materials />-->
 		<link name="base_0">
 			<inertial>
@@ -205,6 +205,6 @@
 			</visual>
 		</link>
-		<xacro:dsr_transmission />
-		<xacro:dsr_gazebo namespace="${namespace}" />
+<!--		<xacro:dsr_transmission />-->
+<!--		<xacro:dsr_gazebo namespace="${namespace}" />-->
 	</xacro:macro>
 </robot>
