Commit message: add tcp to doosan

File: dsr_description/xacro/m1013.urdf.xacro (robot description, xacro)
@@ -16,4 +16,5 @@
      <xacro:include filename="$(find dsr_description)/xacro/robotiq_2f.urdf.xacro" />
   </xacro:if>
+  <link name="tcp" />
   <!-- World fixed joint-->
   <joint name="world_fixed" type="fixed">
@@ -22,3 +23,9 @@
     <child link="base_0"/>
   </joint>
+  <!-- TCP fixed joint-->
+  <joint name="tcp_fixed" type="fixed">
+    <origin xyz="0 0 0.1" rpy="0 -1.57075 0"/>
+    <parent link="link6"/>
+    <child link="tcp"/>
+  </joint>
 </robot>

Commit message: change initial ref to map

File: dsr_description/xacro/m1013.urdf.xacro (robot description, xacro)
@@ -19,4 +19,9 @@
      <xacro:include filename="$(find dsr_description)/xacro/robotiq_2f.urdf.xacro" />
   </xacro:if>
+<<<<<<< Updated upstream
+=======
+  <link name="tcp" />
+  <link name="map" />
+>>>>>>> Stashed changes
   <!-- World fixed joint-->
   <joint name="world_fixed" type="fixed">
@@ -25,3 +30,18 @@
     <child link="base_0"/>
   </joint>
+<<<<<<< Updated upstream
+=======
+    <!-- World fixed joint-->
+    <joint name="map_planar" type="planar">
+      <origin xyz="0 0 0.76" rpy="0 0 0"/>
+      <parent link="map"/>
+      <child link="world"/>
+    </joint>
+  <!-- TCP fixed joint-->
+  <joint name="tcp_fixed" type="fixed">
+    <origin xyz="0 0 0.1" rpy="0 -1.57075 0"/>
+    <parent link="link6"/>
+    <child link="tcp"/>
+  </joint>
+>>>>>>> Stashed changes
 </robot>

Commit message: change moveit refermce to map for using in mir

File: dsr_description/xacro/m1013.urdf.xacro (robot description, xacro)
@@ -26,5 +26,5 @@
     <!-- World fixed joint-->
     <joint name="map_planar" type="planar">
-      <origin xyz="0 0 0.76" rpy="0 0 0"/>
+      <origin xyz="0 0 0" rpy="0 0 0"/>
       <parent link="map"/>
       <child link="world"/>

Commit message: link doosan to map frame

File: dsr_description/xacro/m1013.urdf.xacro (robot description, xacro)
@@ -5,7 +5,10 @@
   <xacro:property name="cr" value="$(arg color)"/>
   <xacro:property name="gr" value="$(arg gripper)"/>
+<<<<<<< Updated upstream
   	<!-- <xacro:include filename="$(find dsr_description)/config/macro.gazebo.xacro" /> -->
 	<xacro:include filename="$(find dsr_description)/config/macro.transmission.xacro" />
 	<xacro:include filename="$(find dsr_description)/config/macro.materials.xacro" />
+=======
+>>>>>>> Stashed changes
   <xacro:if value="${cr == 'white'}">
      <xacro:include filename="$(find dsr_description)/xacro/macro.m1013.white.xacro" />
@@ -19,4 +22,9 @@
      <xacro:include filename="$(find dsr_description)/xacro/robotiq_2f.urdf.xacro" />
   </xacro:if>
+<<<<<<< Updated upstream
+=======
+  <link name="tcp" />
+  <link name="map" />
+>>>>>>> Stashed changes
   <!-- World fixed joint-->
   <joint name="world_fixed" type="fixed">
@@ -25,3 +33,18 @@
     <child link="base_0"/>
   </joint>
+<<<<<<< Updated upstream
+=======
+    <!-- World fixed joint-->
+    <joint name="map_planar" type="planar">
+      <origin xyz="0 0 0.76" rpy="0 0 0"/>
+      <parent link="map"/>
+      <child link="world"/>
+    </joint>
+  <!-- TCP fixed joint-->
+  <joint name="tcp_fixed" type="fixed">
+    <origin xyz="0 0 0.1" rpy="0 -1.57075 0"/>
+    <parent link="link6"/>
+    <child link="tcp"/>
+  </joint>
+>>>>>>> Stashed changes
 </robot>

Commit message: add camera and tool collisions

File: dsr_description/xacro/m1013.urdf.xacro (robot description, xacro)
@@ -16,6 +16,6 @@
      <xacro:include filename="$(find dsr_description)/xacro/robotiq_2f.urdf.xacro" />
   </xacro:if>
-  <link name="tcp" />
-  <link name="map" />
+  <!-- <link name="tcp" /> -->
+  <!-- <link name="map" /> -->
   <!-- World fixed joint-->
   <joint name="world_fixed" type="fixed">
@@ -25,14 +25,26 @@
   </joint>
     <!-- World fixed joint-->
-    <joint name="map_planar" type="planar">
+    <!-- <joint name="map_planar" type="planar">
       <origin xyz="0 0 0" rpy="0 0 0"/>
       <parent link="map"/>
       <child link="world"/>
-    </joint>
+    </joint> -->
   <!-- TCP fixed joint-->
-  <joint name="tcp_fixed" type="fixed">
+  <!-- <joint name="tcp_fixed" type="fixed">
     <origin xyz="0 0 0.1" rpy="0 -1.57075 0"/>
     <parent link="link6"/>
     <child link="tcp"/>
+  </joint> -->
+  <xacro:include filename="$(find azure_kinect_ros_driver)/urdf/azure_kinect.urdf.xacro" />
+  <joint name="camera_fixed" type="fixed">
+    <origin xyz="-0.05 0 0.1" rpy="0 -1.57 0"/>
+    <parent link="link6"/>
+    <child link="camera_base"/>
+  </joint>
+  <xacro:include filename="$(find vacuum)/urdf/vacuum.urdf"/>
+  <joint name="vacuum_fixed" type="fixed">
+    <origin xyz="0 0 0" rpy="1.57 0 0"/>
+    <parent link="link6"/>
+    <child link="vacuum_base_link"/>
   </joint>
 </robot>
