Commit message: add avoidance

File: dsr_description/xacro/macro.m1013.white.xacro (robot description, xacro)
@@ -27,5 +27,5 @@
 			<origin rpy="0 0 0" xyz="0 0 0.1525" />
 			<axis xyz="0 0 1" />
-			<limit effort="346" lower="-6.2832" upper="6.2832" velocity="2.0944"/>
+			<limit effort="346" lower="-1.5708" upper="0.785398" velocity="2.0944"/>
 			<dynamics friction="0" />
 		</joint>
@@ -122,5 +122,5 @@
 			<origin rpy="1.571 0 0" xyz="0 -0.559 0" />
 			<axis xyz="0 0 1" />
-			<limit effort="50" lower="-6.2832" upper="6.2832" velocity="3.927"/>
+			<limit effort="50" lower="0" upper="6.2832" velocity="3.927"/>
 			<dynamics friction="0" />
 		</joint>
@@ -157,5 +157,5 @@
 			<origin rpy="-1.571 0 0" xyz="0 0 0" />
 			<axis xyz="0 0 1" />
-			<limit effort="50" lower="-6.2832" upper="6.2832" velocity="3.927"/>
+			<limit effort="50" lower="-1.74533" upper="1.57" velocity="3.927"/>
 			<dynamics friction="0" />
 		</joint>
@@ -174,4 +174,10 @@
                 </geometry>
             </collision>
+			<collision>
+                <origin rpy="0 0 0" xyz="0 0 0.15" />
+                <geometry>
+                    <cylinder radius="0.08" length="0.15"/>
+                </geometry>
+            </collision>
 			<visual>
 				<origin rpy="0 0 0" xyz="0 0 0" />
@@ -187,5 +193,5 @@
 			<origin rpy="1.571 0 0" xyz="0 -0.121 0" />
 			<axis xyz="0 0 1" />
-			<limit effort="50" lower="-6.2832" upper="6.2832" velocity="3.927"/>
+			<limit effort="50" lower="-3.1415" upper="0" velocity="3.927"/>
 			<dynamics friction="0" />
 		</joint>
